File: Schematic/ATRescueBoard/ATRescueBoard.brd (EAGLE design)
At the start: 44.7 x 53.3 mm, 19 parts, among them IC1 ATMEGA, Q1 2N3904, U1 TINY85-20-DIP

Commit message: Completed first version of schematic and board
Parts:
- removed IC1: ATMEGA, avr-4:DIL28-3
- added MCU2: ATTINY84ATTINY84-20PU, SparkFun-DigitalIC:DIL14
- added R6: 560, rcl:0309/12
- LED1, LED2: device mightyohm:LED3MM -> mightyohm:LED5MM
- MCU1: value ATTINY84ATTINY84-20PU -> ATMEGA; device SparkFun-DigitalIC:DIL14 -> avr-4:DIL28-3
- R1: device rcl:0207/10 -> rcl:0204/7
- R3, R4: device rcl:0204/5 -> rcl:0309/12
- R5: value 560 -> 4K7; device rcl:0204/5 -> rcl:0204/7
- moved R2 25.7 mm to (37.1, 7.62)
- moved C1 25.2 mm to (21.6, 28.7), turned to 90 degrees
- moved R5 20.5 mm to (24.9, 11.2)
- moved MCU1 16.3 mm to (24.4, 41.1)
- moved R1 14.0 mm to (24.9, 7.62)
- moved R4 10.9 mm to (16.3, 18.8)
- moved R3 10.8 mm to (16.3, 22.6)
- moved Q1 8.89 mm to (13.0, 7.62)
- moved TP1 6.99 mm to (2.79, 23.6)
- moved SW1 5.61 mm to (3.05, 31.2)
- moved POWER 1.26 mm to (16.8, 2.54)
- renumbered J1 to DIG0_7, J2 to ANA_IN, J3 to DIG8_13, U1 to MCU3
Connections:
- net !OE: now also MCU1.4; no longer IC1.4
- net !WR: now also MCU1.5; no longer IC1.5
- net 12V_EN: now also R6.1
- net 5V: now also R6.2
- net BS1/SCI: now also MCU1.6, MCU2.2; no longer IC1.6, MCU1.2
- net BS2: now also MCU1.25; no longer IC1.25
- net DATA0: now also MCU1.14; no longer IC1.14
- net DATA1: now also MCU1.15; no longer IC1.15
- net DATA2: now also MCU1.16; no longer IC1.16
- net DATA3: now also MCU1.17; no longer IC1.17
- net DATA4: now also MCU1.18; no longer IC1.18
- net DATA5: now also MCU1.19; no longer IC1.19
- net DATA6: now also MCU1.23; no longer IC1.23
- net DATA7: now also MCU1.24; no longer IC1.24
- net GND: now also MCU1.22, MCU1.8, MCU2.11, MCU2.12, MCU2.13, MCU2.14; no longer IC1.22, IC1.8, MCU1.11, MCU1.12, MCU1.13, MCU1.14
- net PAGEL: now also MCU1.13; no longer IC1.13
- net RDY/SDO: now also MCU1.3, MCU2.9; no longer IC1.3, MCU1.9
- net RESET: now also MCU1.1, MCU2.4; no longer IC1.1, MCU1.4
- net VCC: now also MCU1.20, MCU1.7, MCU2.1; no longer IC1.20, IC1.7, MCU1.1
- net XA0/SII: now also MCU1.11, MCU2.8; no longer IC1.11, MCU1.8
- net XA1/SDI: now also MCU1.12, MCU2.7; no longer IC1.12, MCU1.7
- net XTAL1: now also MCU1.9; no longer IC1.9
Routing:
- net GND: track 0.00 -> 123.6 mm
- net VCC: track 0.00 -> 71.8 mm
- net RDY/SDO: track 0.00 -> 67.0 mm
- net 12V_SW: track 0.00 -> 57.9 mm
- net BS1/SCI: track 0.00 -> 47.4 mm
- net !GO: track 0.00 -> 47.1 mm
- net RESET: track 0.00 -> 44.0 mm
- net 12V_EN: track 0.00 -> 43.4 mm
- net XA0/SII: track 0.00 -> 43.3 mm
- net XTAL1: track 0.00 -> 39.7 mm
- net 5V: track 0.00 -> 39.7 mm
- net XA1/SDI: track 0.00 -> 37.4 mm
- net PAGEL: track 0.00 -> 37.2 mm
- net N$21: track 0.00 -> 31.5 mm
- net N$7: track 0.00 -> 20.5 mm
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- removed copper zone on layer 16, net GND
Other:
- board text added: "00"
- board text added: "01"
- board text added: "02"
- board text added: "03"
- board text added: "04"
- board text added: "05"
- board text added: "06"
- board text added: "07"
- board text added: "08"
- board text added: "09"
- board text added: "10"
- board text added: "11"
- board text added: "12"
- board text added: "13"
- board text added: "3.3V"
- board text added: "5V"
- board text added: "A0"
- board text added: "A1"
- board text added: "A2"
- board text added: "A3"
- board text added: "A4"
- board text added: "A5"
- board text added: "IOREF"
- board text added: "VIN"
- board text removed: "011411"
- board text removed: "JSK"
