File: Schematic/ATRescueBoard/ATRescueBoard.sch (EAGLE design)
At the start: 18 parts, among them IC1 ATMEGA, Q1 2N3904, U1 TINY85-20-DIP

Commit message: Completed first version of schematic and board
Parts:
- removed IC1: ATMEGA, avr-4:MEGA48/88/168-PU
- added MCU2: ATTINY84ATTINY84-20PU, SparkFun-DigitalIC:ATTINY84ATTINY84-20PU
- added R6: 560, rcl:R-US_0309/12
- LED1, LED2: device mightyohm:LED3MM -> mightyohm:LED5MM
- MCU1: value ATTINY84ATTINY84-20PU -> ATMEGA; device SparkFun-DigitalIC:ATTINY84ATTINY84-20PU -> avr-4:MEGA48/88/168-PU
- R1: device rcl:R-US_0207/10 -> rcl:R-US_0204/7
- R3, R4: device rcl:R-US_0204/5 -> rcl:R-US_0309/12
- R5: value 560 -> 4K7; device rcl:R-US_0204/5 -> rcl:R-US_0204/7
- renumbered J1 to DIG0_7, J2 to ANA_IN, J3 to DIG8_13, U1 to MCU3
Connections:
- net !OE: now also MCU1.PD2(INT0/PCINT18); no longer IC1.PD2(INT0/PCINT18)
- net !WR: now also MCU1.PD3(INT1/OC2B/PCINT19); no longer IC1.PD3(INT1/OC2B/PCINT19)
- net 12V_EN: now also R6.1
- net 5V: now also R6.2
- net BS1/SCI: now also MCU1.PD4(T0/XCK/PCINT20), MCU2.(PCINT8/XTAL1/CLKI)PB0; no longer IC1.PD4(T0/XCK/PCINT20), MCU1.(PCINT8/XTAL1/CLKI)PB0
- net BS2: now also MCU1.PC2(ADC2/PCINT10); no longer IC1.PC2(ADC2/PCINT10)
- net DATA0: now also MCU1.PB0(ICP1/CLKO/PCINT0); no longer IC1.PB0(ICP1/CLKO/PCINT0)
- net DATA1: now also MCU1.PB1(OC1A/PCINT1); no longer IC1.PB1(OC1A/PCINT1)
- net DATA2: now also MCU1.PB2(SS/OC1B/PCINT2); no longer IC1.PB2(SS/OC1B/PCINT2)
- net DATA3: now also MCU1.PB3(MOSI/OC2A/PCINT3); no longer IC1.PB3(MOSI/OC2A/PCINT3)
- net DATA4: now also MCU1.PB4(MISO/PCINT4); no longer IC1.PB4(MISO/PCINT4)
- net DATA5: now also MCU1.PB5(SCK/PCINT5); no longer IC1.PB5(SCK/PCINT5)
- net DATA6: now also MCU1.PC0(ADC0/PCINT8); no longer IC1.PC0(ADC0/PCINT8)
- net DATA7: now also MCU1.PC1(ADC1/PCINT9); no longer IC1.PC1(ADC1/PCINT9)
- net GND: now also MCU1.AGND, MCU1.GND@1, MCU2.(PCINT0/AREF/ADC0)PA0, MCU2.(PCINT1/AIN0/ADC1)PA1, MCU2.(PCINT2/AIN1/ADC2)PA2, MCU2.GND; no longer IC1.AGND, IC1.GND@1, MCU1.(PCINT0/AREF/ADC0)PA0, MCU1.(PCINT1/AIN0/ADC1)PA1, MCU1.(PCINT2/AIN1/ADC2)PA2, MCU1.GND
- net PAGEL: now also MCU1.PD7(AIN1/PCINT23); no longer IC1.PD7(AIN1/PCINT23)
- net RDY/SDO: now also MCU1.PD1(TXD/PCINT17), MCU2.(PCINT4/T1/SCL/USCK/ADC4)PA4; no longer IC1.PD1(TXD/PCINT17), MCU1.(PCINT4/T1/SCL/USCK/ADC4)PA4
- net RESET: now also MCU1.PC6(/RESET/PCINT14), MCU2.(PCINT11/~RESET/DW)PB3; no longer IC1.PC6(/RESET/PCINT14), MCU1.(PCINT11/~RESET/DW)PB3
- net VCC: now also MCU1.AVCC, MCU1.VCC@1, MCU2.VCC; no longer IC1.AVCC, IC1.VCC@1, MCU1.VCC
- net XA0/SII: now also MCU1.PD5(T1/OC0B/PCINT21), MCU2.(PCINT5/OC1B/MISO/DO/ADC5)PA5; no longer IC1.PD5(T1/OC0B/PCINT21), MCU1.(PCINT5/OC1B/MISO/DO/ADC5)PA5
- net XA1/SDI: now also MCU1.PD6(AIN0/OC0A/PCINT22), MCU2.(PCINT6/OC1A/SDA/MOSI/ADC6)PA6; no longer IC1.PD6(AIN0/OC0A/PCINT22), MCU1.(PCINT6/OC1A/SDA/MOSI/ADC6)PA6
- net XTAL1: now also MCU1.PB6(XTAL1/TOSC1/PCINT6); no longer IC1.PB6(XTAL1/TOSC1/PCINT6)
